File: Schematic_and_Board/FanControl.sch (EAGLE design)
At the start: 45 parts, among them J1 POWER_JACKSLT, Q1 VP3203, Q2 VP3203, T1 2N3904, T2 2N3904, U1 ARDUINO_MINI, U2 LCD-16X2SILK

Commit message: Update Schematic and Board to correct these two errors:
Connections:
- net GND: now also J1.GNDBREAK
- net N$11: now also Q1.D; no longer Q1.S
- net N$15: now also Q2.D; no longer Q2.S
- net V12: now also Q1.S, Q2.S; no longer Q1.D, Q2.D
Other:
- moved on the sheet: Q1, Q2
Changed lines of the file:
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@@
 <instance part="T1" gate="G1" x="45.72" y="99.06"/>
 <instance part="R12" gate="G$1" x="48.26" y="86.36" rot="R270"/>
-<instance part="Q1" gate="G$1" x="66.04" y="109.22"/>
+<instance part="Q1" gate="G$1" x="66.04" y="104.14" rot="MR180"/>
 <instance part="POT1" gate="G$1" x="116.84" y="170.18"/>
 <instance part="D1" gate="1" x="73.66" y="86.36" rot="R90"/>
@@
 <instance part="T2" gate="G1" x="45.72" y="40.64"/>
 <instance part="R15" gate="G$1" x="48.26" y="27.94" rot="R270"/>
-<instance part="Q2" gate="G$1" x="66.04" y="50.8"/>
+<instance part="Q2" gate="G$1" x="66.04" y="45.72" rot="MR180"/>
 <instance part="D2" gate="1" x="73.66" y="27.94" rot="R90"/>
 <instance part="L2" gate="G$1" x="93.98" y="40.64" rot="R90"/>
@@
 <junction x="48.26" y="121.92"/>
 <label x="43.18" y="121.92" size="0.8128" layer="95" rot="R180" xref="yes"/>
-<wire x1="73.66" y1="121.92" x2="73.66" y2="111.76" width="0.1524" layer="91"/>
-<pinref part="Q1" gate="G$1" pin="D"/>
-<wire x1="73.66" y1="111.76" x2="71.12" y2="111.76" width="0.1524" layer="91"/>
+<wire x1="73.66" y1="121.92" x2="73.66" y2="106.68" width="0.1524" layer="91"/>
+<pinref part="Q1" gate="G$1" pin="S"/>
+<wire x1="71.12" y1="106.68" x2="73.66" y2="106.68" width="0.1524" layer="91"/>
 </segment>
 <segment>
@@
 <junction x="48.26" y="63.5"/>
 <label x="43.18" y="63.5" size="0.8128" layer="95" rot="R180" xref="yes"/>
-<wire x1="73.66" y1="63.5" x2="73.66" y2="53.34" width="0.1524" layer="91"/>
-<pinref part="Q2" gate="G$1" pin="D"/>
-<wire x1="73.66" y1="53.34" x2="71.12" y2="53.34" width="0.1524" layer="91"/>
+<wire x1="73.66" y1="63.5" x2="73.66" y2="48.26" width="0.1524" layer="91"/>
+<pinref part="Q2" gate="G$1" pin="S"/>
+<wire x1="71.12" y1="48.26" x2="73.66" y2="48.26" width="0.1524" layer="91"/>
 </segment>
 </net>
@@
 <junction x="101.6" y="157.48"/>
 <pinref part="J1" gate="G$1" pin="GND"/>
-<wire x1="38.1" y1="175.26" x2="50.8" y2="175.26" width="0.1524" layer="91"/>
+<wire x1="38.1" y1="175.26" x2="40.64" y2="175.26" width="0.1524" layer="91"/>
+<wire x1="40.64" y1="175.26" x2="50.8" y2="175.26" width="0.1524" layer="91"/>
 <wire x1="50.8" y1="175.26" x2="50.8" y2="157.48" width="0.1524" layer="91"/>
 <wire x1="50.8" y1="157.48" x2="78.74" y2="157.48" width="0.1524" layer="91"/>
@@
 <pinref part="U$1" gate="G$1" pin="GND"/>
 <pinref part="POT1" gate="G$1" pin="1"/>
+<pinref part="J1" gate="G$1" pin="GNDBREAK"/>
+<wire x1="38.1" y1="177.8" x2="40.64" y2="177.8" width="0.1524" layer="91"/>
+<wire x1="40.64" y1="177.8" x2="40.64" y2="175.26" width="0.1524" layer="91"/>
+<junction x="40.64" y="175.26"/>
 </segment>
 <segment>
@@
 <segment>
 <pinref part="R10" gate="G$1" pin="1"/>
-<wire x1="48.26" y1="109.22" x2="48.26" y2="106.68" width="0.1524" layer="91"/>
-<wire x1="48.26" y1="106.68" x2="60.96" y2="106.68" width="0.1524" layer="91"/>
 <pinref part="T1" gate="G1" pin="C"/>
 <wire x1="48.26" y1="104.14" x2="48.26" y2="106.68" width="0.1524" layer="91"/>
+<pinref part="Q1" gate="G$1" pin="G"/>
+<wire x1="48.26" y1="106.68" x2="48.26" y2="109.22" width="0.1524" layer="91"/>
+<wire x1="60.96" y1="106.68" x2="48.26" y2="106.68" width="0.1524" layer="91"/>
 <junction x="48.26" y="106.68"/>
-<pinref part="Q1" gate="G$1" pin="G"/>
 </segment>
 </net>
@@
 <net name="N$11" class="0">
 <segment>
-<pinref part="Q1" gate="G$1" pin="S"/>
-<wire x1="71.12" y1="106.68" x2="73.66" y2="106.68" width="0.1524" layer="91"/>
 <pinref part="D1" gate="1" pin="C"/>
-<wire x1="73.66" y1="106.68" x2="73.66" y2="99.06" width="0.1524" layer="91"/>
+<wire x1="73.66" y1="101.6" x2="73.66" y2="99.06" width="0.1524" layer="91"/>
 <pinref part="L1" gate="G$1" pin="1"/>
 <wire x1="73.66" y1="99.06" x2="73.66" y2="88.9" width="0.1524" layer="91"/>
 <wire x1="86.36" y1="99.06" x2="73.66" y2="99.06" width="0.1524" layer="91"/>
 <junction x="73.66" y="99.06"/>
+<pinref part="Q1" gate="G$1" pin="D"/>
+<wire x1="71.12" y1="101.6" x2="73.66" y2="101.6" width="0.1524" layer="91"/>
 </segment>
 </net>
@@
 <segment>
 <pinref part="R13" gate="G$1" pin="1"/>
-<wire x1="48.26" y1="50.8" x2="48.26" y2="48.26" width="0.1524" layer="91"/>
-<wire x1="48.26" y1="48.26" x2="60.96" y2="48.26" width="0.1524" layer="91"/>
 <pinref part="T2" gate="G1" pin="C"/>
 <wire x1="48.26" y1="45.72" x2="48.26" y2="48.26" width="0.1524" layer="91"/>
+<pinref part="Q2" gate="G$1" pin="G"/>
+<wire x1="48.26" y1="48.26" x2="48.26" y2="50.8" width="0.1524" layer="91"/>
+<wire x1="60.96" y1="48.26" x2="48.26" y2="48.26" width="0.1524" layer="91"/>
 <junction x="48.26" y="48.26"/>
-<pinref part="Q2" gate="G$1" pin="G"/>
 </segment>
 </net>
@@
 <net name="N$15" class="0">
 <segment>
-<pinref part="Q2" gate="G$1" pin="S"/>
-<wire x1="71.12" y1="48.26" x2="73.66" y2="48.26" width="0.1524" layer="91"/>
 <pinref part="D2" gate="1" pin="C"/>
-<wire x1="73.66" y1="48.26" x2="73.66" y2="40.64" width="0.1524" layer="91"/>
+<wire x1="73.66" y1="43.18" x2="73.66" y2="40.64" width="0.1524" layer="91"/>
 <pinref part="L2" gate="G$1" pin="1"/>
 <wire x1="73.66" y1="40.64" x2="73.66" y2="30.48" width="0.1524" layer="91"/>
 <wire x1="86.36" y1="40.64" x2="73.66" y2="40.64" width="0.1524" layer="91"/>
 <junction x="73.66" y="40.64"/>
-</segment>
-</net>
+<pinref part="Q2" gate="G$1" pin="D"/>
+<wire x1="71.12" y1="43.18" x2="73.66" y2="43.18" width="0.1524" layer="91"/>
+</segment>
+</net>
